File: PX4Node_mini_V0_1_1.sch (EAGLE design)
At the start: 127 parts, among them J2 DF13-4P-1.25V, J201 DF13C-6P-1.25V, J202 DF13C-6P-1.25V, J203 DF13C-6P-1.25V, J3 DF13C-4P-1.25V, J302 DF13C-4P-1.25V, J401 DF13C-4P-1.25V, J403 DF13C-7P-1.25V, J405 DF13C-4P-1.25V, J802 DF13C-3P-1.25V, M3_MOUNT1101 MOUNT-HOLE3.1MM, M3_MOUNT1102 MOUNT-HOLE3.1MM, M3_MOUNT1103 MOUNT-HOLE3.1MM, M3_MOUNT1104 MOUNT-HOLE3.1MM, U101 STM32F4X7VX, U2 MAX3051, U401 MAX3051, X101 3.2x2.5 mm / 24 MHz / 15 ppm

Commit message: Some tweaks
Parts:
- added SJ3: SOLDERJUMPERNO, SparkFun-Passives:SOLDERJUMPERNO
Connections:
- new net 5V_CAN_CONN: L403.P$1, L7.P$1, SJ3.2
- net VDD_5V_PERIPH: now also SJ3.1; no longer L403.P$1, L7.P$1
Changed lines of the file:
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@@
 <layer number="91" name="Nets" color="2" fill="1" visible="yes" active="yes"/>
 <layer number="92" name="Busses" color="1" fill="1" visible="yes" active="yes"/>
-<layer number="93" name="Pins" color="2" fill="1" visible="yes" active="yes"/>
+<layer number="93" name="Pins" color="2" fill="1" visible="no" active="yes"/>
 <layer number="94" name="Symbols" color="4" fill="1" visible="yes" active="yes"/>
 <layer number="95" name="Names" color="7" fill="1" visible="yes" active="yes"/>
@@
 </part>
 <part name="JP3" library="SparkFun-Connectors" deviceset="M01" device="SMD-4.5X1.5"/>
+<part name="SJ3" library="SparkFun-Passives" deviceset="SOLDERJUMPER" device="NO"/>
 </parts>
 <sheets>
@@
 </instance>
 <instance part="SJ2" gate="1" x="205.74" y="106.68"/>
+<instance part="SJ3" gate="1" x="134.62" y="114.3"/>
 </instances>
 <busses>
@@
 </segment>
 <segment>
-<wire x1="177.8" y1="114.3" x2="139.7" y2="114.3" width="0.1524" layer="91"/>
-<label x="139.7" y="114.3" size="1.27" layer="95" rot="R180" xref="yes"/>
+<label x="124.46" y="114.3" size="1.27" layer="95" rot="R180" xref="yes"/>
+<pinref part="SJ3" gate="1" pin="1"/>
+<wire x1="129.54" y1="114.3" x2="124.46" y2="114.3" width="0.1524" layer="91"/>
+</segment>
+<segment>
+<label x="30.48" y="53.34" size="1.27" layer="95" rot="R180" xref="yes"/>
+<wire x1="66.04" y1="53.34" x2="30.48" y2="53.34" width="0.1524" layer="91"/>
+<pinref part="L4" gate="G$1" pin="P$1"/>
+</segment>
+<segment>
+<wire x1="66.04" y1="114.3" x2="27.94" y2="114.3" width="0.1524" layer="91"/>
+<label x="27.94" y="114.3" size="1.27" layer="95" rot="R180" xref="yes"/>
+<pinref part="L5" gate="G$1" pin="P$1"/>
+</segment>
+</net>
+<net name="5V_CAN_CONN" class="0">
+<segment>
 <pinref part="L7" gate="G$1" pin="P$1"/>
+<wire x1="139.7" y1="114.3" x2="147.32" y2="114.3" width="0.1524" layer="91"/>
+<wire x1="147.32" y1="114.3" x2="177.8" y2="114.3" width="0.1524" layer="91"/>
+<wire x1="147.32" y1="114.3" x2="147.32" y2="121.92" width="0.1524" layer="91"/>
+<wire x1="147.32" y1="121.92" x2="154.94" y2="121.92" width="0.1524" layer="91"/>
+<label x="154.94" y="121.92" size="1.778" layer="95" xref="yes"/>
+<junction x="147.32" y="114.3"/>
+<pinref part="SJ3" gate="1" pin="2"/>
 </segment>
 <segment>
@@
 <pinref part="L403" gate="G$1" pin="P$1"/>
 </segment>
-<segment>
-<label x="30.48" y="53.34" size="1.27" layer="95" rot="R180" xref="yes"/>
-<wire x1="66.04" y1="53.34" x2="30.48" y2="53.34" width="0.1524" layer="91"/>
-<pinref part="L4" gate="G$1" pin="P$1"/>
-</segment>
-<segment>
-<wire x1="66.04" y1="114.3" x2="27.94" y2="114.3" width="0.1524" layer="91"/>
-<label x="27.94" y="114.3" size="1.27" layer="95" rot="R180" xref="yes"/>
-<pinref part="L5" gate="G$1" pin="P$1"/>
-</segment>
-</net>
+</net>
