File: PX4uNode_V0_1_1.sch (EAGLE design)
At the start: 126 parts, among them J2 DF13-4P-1.25V, J201 DF13C-6P-1.25V, J202 DF13C-6P-1.25V, J203 DF13C-6P-1.25V, J3 DF13C-4P-1.25V, J302 DF13C-4P-1.25V, J401 DF13C-4P-1.25V, J403 DF13C-7P-1.25V, J405 DF13C-4P-1.25V, J802 DF13C-3P-1.25V, M3_MOUNT1101 MOUNT-HOLE3.1MM, M3_MOUNT1102 MOUNT-HOLE3.1MM, M3_MOUNT1103 MOUNT-HOLE3.1MM, M3_MOUNT1104 MOUNT-HOLE3.1MM, U101 STM32F4X7VX, U2 MAX3051, U401 MAX3051, X101 3.2x2.5 mm / 24 MHz / 15 ppm

Commit message: Added uNode, Removed old versions of mNode
Parts:
- removed C1, C10, C8, C9: 22uF, SparkFun-Capacitors:22UF-16V-20%-(1210)
- removed C103: 8p, pixhawk2:CAP0402
- removed C12, C6, C609, C612, C7: 0u1, pixhawk2:CAP0402
- removed FMU-BOOT0: PAD.04, pixhawk2:PAD.04
- removed J1: (no value), PX4lite:SERVO_HEADER-3X8
- removed J2: DF13-4P-1.25V, con-hirose-df13:DF13-4P-1.25V
- removed J201, J202, J203: DF13C-6P-1.25V, con-hirose-df13:DF13-6P-1.25V
- removed J3, J302, J401, J405: DF13C-4P-1.25V, con-hirose-df13:DF13-4P-1.25V
- removed J403: DF13C-7P-1.25V, con-hirose-df13:DF13-7P-1.25V
- removed J802: DF13C-3P-1.25V, con-hirose-df13:DF13-3P-1.25V
- removed L2, L3, L6: NUF8402MN, PX4lite:NUF8402MN
- removed L4, L5, L7: KNH16C104DA5TS, pixhawk2:KNH16C104DA5TS
- removed R1: 1K5, pixhawk2:RESISTOR0402-RES
- removed R4, R409: 120R, pixhawk2:RESISTOR0402-RES
- removed R608: 1K, pixhawk2:RESISTOR0402-RES
- removed R609, R610: 10K/0.1%, pixhawk2:RESISTOR0402-RES
- removed R611: 10K, pixhawk2:RESISTOR0402-RES
- removed S601: RESET, pixhawk2:SWITCH-MOMENTARY-2
- removed SJ1, SJ2: SOLDERJUMPERTRACE, SparkFun-Passives:SOLDERJUMPERTRACE
- removed U$1: HEADER-3X1BOARDEDGE-SHORT, PX4lite:HEADER-3X1BOARDEDGE-SHORT
- removed U$14: HEADER-3X1RA, PX4lite:HEADER-3X1RA
- removed U$4: PESD0402-140, pixhawk2:DIODE-TVS
- removed U$604: BQ24315, pixhawk2:BQ24315
- removed U$605: MIC5332, pixhawk2:MIC5332
- removed U2: MAX3051, pixhawk2:MAX3051MAX3051EKA
- added BOOT: PAD.04, pixhawk2:PAD.04
- added C101: 8p, pixhawk2:CAP0402
- added C201, C711, C712, C714, C717: 0u1, pixhawk2:CAP0402
- added C701: 2u2, pixhawk2:CAP0603
- added C703: 10n, pixhawk2:CAP0402
- added C705, C708: 1u0, pixhawk2:CAP0603
- added C706: 10u/10V, pixhawk2:CAP0805
- added D701: MSS1P4-M3, pixhawk2:DIODE-SCHOTTKY_MSMP
- added J1001: (no value), PX4lite:SERVO_HEADER-3X8
- added JP10, JP9: (no value), SparkFun-Connectors:M03PTH
- added JP1001, JP1002, JP701, JP702: M01SMD-4.5X1.5, SparkFun-Connectors:M01SMD-4.5X1.5
- added JP11, JP6, JP7, JP8: (no value), SparkFun-Connectors:M04PTH
- added JP1102, JP1103, JP1104: FIDUCIAL1.5X3, pixhawk2:FIDUCIAL1.5X3
- added JP12: (no value), SparkFun-Connectors:M03X22X3_SILK_SM
- added JP201: JUMPER-3SMD, SparkFun-Passives:JUMPER-3SMD
- added JP202: (no value), SparkFun-Passives:JUMPER-2SMD-NO
- added JP4: (no value), SparkFun-Connectors:M07
- added JP901: M02PTH3, SparkFun-Connectors:M02PTH3
- added L204, L205, L401, L404, L405, L406: KNH16C104DA5TS, PX4lite:KNH16C104DA5TS
- added R1001, R804: 220R, pixhawk2:RESISTOR0402-RES
- added R404: 1K5, pixhawk2:RESISTOR0402-RES
- added R405, R406, R708: 10K/0.1%, pixhawk2:RESISTOR0402-RES
- added R702, R709: 10K, pixhawk2:RESISTOR0402-RES
- added R706: 1K, pixhawk2:RESISTOR0402-RES
- added S701: RESET, pixhawk2:SWITCH-MOMENTARY-2
- added SJ401: SOLDERJUMPERNO, SparkFun-Passives:SOLDERJUMPERNO
- added SJ402, SJ403: SOLDERJUMPERNC2, SparkFun-Passives:SOLDERJUMPERNC2
- added U$204, U$205, U$402, U$801: PESD0402-140, pixhawk2:DIODE-TVS
- added U$703: BQ24315, PX4lite:BQ24315
- added U402: MAX3051, pixhawk2:MAX3051MAX3051EKA
- added X1: USB-MICROB, pixhawk2:USB-MICROB
- C601: value 2u2 -> 22uF; device pixhawk2:CAP0603 -> SparkFun-Capacitors:22UF-16V-20%-(1210); PARTNO C1608Y5V1C225Z -> (none)
- C602: value 10n -> 0u1; PARTNO CC0402KRX7R7BB103 -> CC0402ZRY5V7BB104
- C603: value 1u0 -> 0u1; device pixhawk2:CAP0603 -> pixhawk2:CAP0402; PARTNO CC0603ZRY5V7BB105 -> CC0402ZRY5V7BB104
- C604: value 10u/10V -> 0u1; device pixhawk2:CAP0805 -> pixhawk2:CAP0402; PARTNO CC0805ZKY5V6BB106 -> CC0402ZRY5V7BB104
- C605: value 1u0 -> 22uF; device pixhawk2:CAP0603 -> SparkFun-Capacitors:22UF-16V-20%-(1210); PARTNO CC0603ZRY5V7BB105 -> (none)
- C606, C607: value 0u1 -> 22uF; device pixhawk2:CAP0402 -> SparkFun-Capacitors:22UF-16V-20%-(1210); PARTNO CC0402ZRY5V7BB104 -> (none)
- D901: BOM (none) -> EXCLUDE
- D902, D903: PARTNO (none) -> B340A
- JP1, JP2: value FIDUCIAL1.5X3 -> (none); device pixhawk2:FIDUCIAL1.5X3 -> SparkFun-Connectors:M03X22X3_SILK_SM; BOM EXCLUDE -> (none); PARTNO * -> (none)
- JP5: value M02PTH3 -> (none); device SparkFun-Connectors:M02PTH3 -> SparkFun-Connectors:M04PTH
- L201, L202, L402: value KNH16C104DA5TS -> NUF8402MN; device pixhawk2:KNH16C104DA5TS -> PX4lite:NUF8402MN; PARTNO KNH16C104DA5TS -> (none)
- L203, L403: device pixhawk2:KNH16C104DA5TS -> PX4lite:KNH16C104DA5TS
- R1002: value 10K -> 220R; PARTNO RC0402FR-0710KL -> RC0402FR-07220RL
- R407, R408: value 10K/0.1% -> 120R; PARTNO ERA-2AEB103X -> RC0402FR-07120RL
- R704: value 25K -> 47K; PARTNO RMCF0402FT25K5 -> RMCF0402FT47K
- R707: value 220R -> 10K/0.1%; PARTNO RC0402FR-07220RL -> ERA-2AEB103X
- U$201: value PESD0402-140 -> HEADER-3X1RA; device pixhawk2:DIODE-TVS -> PX4lite:HEADER-3X1RA; PARTNO PESD0402-140 -> (none)
- U$202: value PESD0402-140 -> 74LVC2GU04; device pixhawk2:DIODE-TVS -> pixhawk2:74LVC2GU04; PARTNO PESD0402-140 -> 74LVC2GU04
- U$701: value PESD0402-140 -> MIC5332; device pixhawk2:DIODE-TVS -> pixhawk2:MIC5332; PARTNO PESD0402-140 -> MIC5332-SSYMT
- renumbered C1001 to C702, C1002 to C704, C1003 to C707, C1004 to C709, C13 to C301, C14 to C302, C15 to C710, C2 to C403, C3 to C404, C4 to C401, C5 to C503, C505 to C502, C506 to C501, C608 to C713, C610 to C715, C611 to C716, C613 to C718, D1 to D904, D2 to D902, D3 to D901, D5 to D903, L1 to L1001, LED701 to LED801, LED704 to LED802, R102 to R101, R2 to R403, R3 to R803, R5 to R703, R603 to R701, R606 to R704, R607 to R705, R710 to R801, R711 to R805, R713 to R802, R918 to R902, R919 to R903, R922 to R901, U$1002 to U$702, U$15 to U$601, U$16 to L$601, U$2 to U$501, U$3 to U$302, U$5 to U$301, U$7 to U$403
Connections:
- new net 5V_CAN_CONN: L405.P$1, L406.P$1, SJ401.2
- new net N$19: JP1001.1, R1001.1
- new net N$23: JP1002.1, R1002.1
- new net N$5: JP202.1, U$202.2Y
- new net N$9: D701.C, R706.2
- new net VDD_RX_POWER: JP201.2, U$201.2
- net !FMU-LED_AMBER: now also R804.1; no longer R707.1
- net !SPI_EXT_NSS: now also JP4.5; no longer J403.5
- net !VDD_5V_PERIPH_EN: now also U$703.!CE; no longer U$604.!CE
- net !VDD_5V_PERIPH_OC: now also U$703.!FAULT; no longer U$604.!FAULT
- net 5V_S1_FILTERED: now also JP12.2, L203.P$2, U$203.C; no longer J201.1, L201.P$2, U$201.C
- net 5V_S2_FILTERED: now also JP1.2, L204.P$2, U$204.C; no longer J202.1, L202.P$2, U$202.C
- net 5V_S3_FILTERED: now also JP2.2, L205.P$2, U$205.C; no longer J203.1, L203.P$2, U$203.C
- net CAN1_H: now also JP7.2, R408.1, U402.CANH; no longer J405.2, R409.1, U401.CANH
- net CAN1_L: now also JP7.3, SJ403.2, U402.CANL; no longer J405.3, SJ1.2, U401.CANL
- net CAN1_RX: now also U402.DOUT; no longer U401.DOUT
- net CAN1_TX: now also U402.DIN; no longer U401.DIN
- net CAN2_H: now also JP8.2, R407.1, U401.CANH; no longer J3.2, R4.1, U2.CANH
- net CAN2_L: now also JP8.3, SJ402.2, U401.CANL; no longer J3.3, SJ2.2, U2.CANL
- net CAN2_RX: now also U401.DOUT; no longer U2.DOUT
- net CAN2_TX: now also U401.DIN; no longer U2.DIN
- net FMU-!RESET: now also C714.2, JX301-!RESET.S, S701.1, U$701.POR2; no longer C609.2, S601.1, U$605.POR2
- net FMU-BOOT0: now also BOOT.P$1, R709.2; no longer FMU-BOOT0.P$1, R611.2
- net FMU-CH1-PROT: now also J1001-CH1.S; no longer J1-CH1.S
- net FMU-CH10: now also R1002.2
- net FMU-CH8: now also JP202.2
- net FMU-CH9: now also R1001.2
- net FMU-I2C1_SCL: now also L402G$8.P$1, R402.1; no longer L6G$8.P$1, R401.1
- net FMU-I2C1_SDA: now also L402G$7.P$1, R404.1; no longer L6G$7.P$1, R402.1
- net FMU-I2C2_SCL: now also L402G$2.P$1, R401.1; no longer L6G$2.P$1, R1.1
- net FMU-I2C2_SDA: now also L402G$1.P$1; no longer L6G$1.P$1
- net FMU-UART7_RX: now also L202G$5.P$1; no longer L3G$5.P$1
- net FMU-UART7_TX: now also L202G$7.P$1; no longer L3G$6.P$1
- net FMU-UART8_RX: now also U$202.1Y
- net FMU-UART8_TX: now also U$202.2A
- net FMU-USART2_CTS: now also L201G$8.P$1; no longer L2G$8.P$1
- net FMU-USART2_RTS: now also L201G$7.P$1; no longer L2G$7.P$1
- net FMU-USART2_RX: now also L201G$5.P$1; no longer L2G$5.P$1
- net FMU-USART2_TX: now also L201G$6.P$1; no longer L2G$6.P$1
- net FMU-USART3_CTS: now also L201G$2.P$1; no longer L2G$2.P$1
- net FMU-USART3_RTS: now also L201G$1.P$1; no longer L2G$1.P$1
- net FMU-USART3_RX: now also L201G$3.P$1; no longer L2G$3.P$1
- net FMU-USART3_TX: now also L201G$4.P$1; no longer L2G$4.P$1
- net FMU-VDD_3V3: now also C201.1, C705.1, C706.1, C711.1, C712.1, C717.1, D701.A, JP10.1, R404.2, R702.1, U$202.VCC, U$701.VOUT2, U$801.C, U402.VCC; no longer C603.1, C604.1, C606.1, C607.1, C612.1, J802.1, R1.2, R608.2, U$605.VOUT2, U$701.C, U2.VCC
- net FMU_AUX_ADC1: now also R405.1; no longer R408.1
- net FMU_AUX_ADC1_PROT: now also JP9.2, R405.2; no longer R408.2, U$1.2
- net FMU_AUX_ADC2: now also R406.1; no longer R407.1
- net FMU_AUX_ADC2_PROT: now also JP9.1, R406.2; no longer R407.2, U$1.1
- net GND: now also C101.2, C102.1, C201.2, C602.2, C701.2, C703.1, C705.2, C706.2, C708.2, C711.2, C712.2, C714.1, C717.2, J1001-GND.S, JP1.5, JP11.4, JP12.5, JP2.5, JP4.7, JP5.4, JP6.4, JP7.4, JP702.1, JP8.4, JP9.3, JP901.2, L201G$9.GND, L202G$1.P$1, L202G$1.P$2, L202G$2.P$1, L202G$2.P$2, L202G$9.GND, L204.P$3, L205.P$3, L401.P$3, L402G$9.GND, L404.P$3, L405.P$3, L406.P$3, R708.2, R709.1, S701.2, U$201.3, U$202.GND, U$204.A, U$205.A, U$402.A, U$701.GND, U$703.VBAT, U$703.VSS, U$801.A, U402.GND, U402.RS, U402.SHDN, X1.GND; no longer C1.2, C10.2, C102.2, C103.1, C12.2, C6.2, C602.1, C609.1, C612.2, C7.2, C8.2, C9.2, J1-GND.S, J2.4, J201.6, J202.6, J203.6, J3.4, J302.4, J401.4, J403.7, J405.4, JP5.2, L201.P$3, L202.P$3, L2G$9.GND, L3G$9.GND, L4.P$3, L402.P$3, L5.P$3, L6G$9.GND, L7.P$3, R1002.1, R610.2, R611.1, S601.2, U$1.3, U$14.3, U$201.A, U$202.A, U$4.A, U$604.VBAT, U$604.VSS, U$605.GND, U$701.A, U2.GND, U2.RS, U2.SHDN
- net GPIO_EXT_1: now also JP4.6; no longer J403.6
- net MAG_DRDY: now also U$501.DSYNC
- net N$1: now also C102.2; no longer C103.2
- net N$11: now also C703.2, U$701.CSET; no longer C602.2, U$605.CSET
- net N$13: now also R804.2; no longer R707.2
- net N$15: now also J1001-CH8.S; no longer J1-CH8.S
- net N$16: now also J1001-CH7.S; no longer J1-CH7.S
- net N$18: now also L202G$3.P$2, L202G$4.P$2, U$201.1; no longer L3G$3.P$2, L3G$4.P$2, U$14.1
- net N$2: now also C101.1; no longer C102.1
- net N$20: now also JP5.3, L402G$1.P$2; no longer J2.3, L6G$1.P$2
- net N$21: now also JP5.1, L403.P$2, U$401.C; no longer J2.1, L5.P$2, U$4.C
- net N$22: now also R408.2, SJ403.1; no longer R409.2, SJ1.1
- net N$27: now also C603.1; no longer C6.1
- net N$28: now also JP8.1, L405.P$2; no longer J3.1, L7.P$2
- net N$29: now also R407.2, SJ402.1; no longer R4.2, SJ2.1
- net N$33: now also JP6.2, L402G$8.P$2; no longer J401.2, L6G$8.P$2
- net N$34: now also U$703.ILIM; no longer U$604.ILIM
- net N$36: now also J1001-CH6.S; no longer J1-CH6.S
- net N$37: now also JP6.3, L402G$7.P$2; no longer J401.3, L6G$7.P$2
- net N$4: now also JP5.2, L402G$2.P$2; no longer J2.2, L6G$2.P$2
- net N$41: now also JP4.1, L401.P$2; no longer J403.1, L402.P$2
- net N$42: now also JP6.1, L404.P$2, U$402.C; no longer J401.1, L4.P$2, U$401.C
- net N$48: now also JP7.1, L406.P$2; no longer J405.1, L403.P$2
- net N$57: now also JP10.2; no longer J802.2
- net N$68: now also J1001-CH5.S; no longer J1-CH5.S
- net N$77: now also J1001-CH4.S; no longer J1-CH4.S
- net N$78: now also J1001-CH3.S; no longer J1-CH3.S
- net N$79: now also J1001-CH2.S; no longer J1-CH2.S
- net OTG_DM1: now also JP11.3, X1.D-; no longer J302.3
- net OTG_DP1: now also JP11.2, X1.D+; no longer J302.2
- net PPM_INPUT: now also L202G$3.P$1, U$202.1A; no longer L3G$3.P$1
- net SAFETY: now also JP10.3; no longer J802.3
- net SERIAL1_CTS: now also JP12.6, L201G$8.P$2; no longer J201.4, L2G$8.P$2
- net SERIAL1_RTS: now also JP12.4, L201G$7.P$2; no longer J201.5, L2G$7.P$2
- net SERIAL1_RX: now also JP12.3, L201G$5.P$2; no longer J201.3, L2G$5.P$2
- net SERIAL1_TX: now also JP12.1, L201G$6.P$2; no longer J201.2, L2G$6.P$2
- net SERIAL2_CTS: now also JP1.6, L201G$2.P$2; no longer J202.4, L2G$2.P$2
- net SERIAL2_RTS: now also JP1.4, L201G$1.P$2; no longer J202.5, L2G$1.P$2
- net SERIAL2_RX: now also JP1.3, L201G$3.P$2; no longer J202.3, L2G$3.P$2
- net SERIAL2_TX: now also JP1.1, L201G$4.P$2; no longer J202.2, L2G$4.P$2
- net SERIAL3_RX: now also JP2.3, L202G$5.P$2; no longer J203.3, L3G$5.P$2
- net SERIAL3_TX: now also JP2.1, L202G$7.P$2; no longer J203.2, L3G$6.P$2
- net SPEKTRUM_RX: now also L202G$4.P$1; no longer L3G$4.P$1
- net SPI_EXT_MISO: now also JP4.3; no longer J403.3
- net SPI_EXT_MOSI: now also JP4.4; no longer J403.4
- net SPI_EXT_SCK: now also JP4.2; no longer J403.2
- net VBAT: now also JP701.1, R706.1; no longer R608.1
- net VBUS: now also JP11.1, X1.VBUS; no longer J302.1
- net VDD_3V3_SENSORS_EN: now also R702.2; no longer R1002.2
- net VDD_3V3_SPEKTRUM: now also C708.1, JP201.1, U$701.VOUT1; no longer C605.1, U$14.2, U$605.VOUT1
- net VDD_3V3_SPEKTRUM_EN: now also U$701.EN1, U101PORTC_L.PC2; no longer U$605.EN1
- net VDD_5V: now also C604.1, C605.1, C606.1, C607.1, C701.1, R707.2, U$701.EN2, U$701.VIN, U$703.IN; no longer C10.1, C601.1, C7.1, C8.1, C9.1, R609.2, U$604.IN, U$605.EN2, U$605.VIN
- net VDD_5V_PERIPH: now also JP201.3, L204.P$1, L205.P$1, L401.P$1, L404.P$1, SJ401.1, U$703.OUT; no longer L201.P$1, L202.P$1, L4.P$1, L402.P$1, L5.P$1, L7.P$1, U$604.OUT
- net VDD_5V_SENS: now also R707.1, R708.1; no longer R609.1, R610.1
- net VDD_IN: now also C601.1, C602.1; no longer C1.1, C12.1
- net V_EXT: now also JP901.1; no longer JP5.1
- net V_SERVO: now also J1001-VCC.S; no longer J1-VCC.S
Other:
- note added: "Current Limits: I(limit) = 25000 / R(ilim) 25K = 1A, 16K5 = 1.5A, 47K ~500mA"
- note added: "DO NOT FIT"
- note added: "FMU Power FMU Reset Battery backup Peripheral power control"
- note added: "FMU Serial ports SBUS interface Spektrum interface"
- note added: "FMU SoC Ports"
- note added: "FMU-CH10 changed to Spektrum 3v3 EN"
- note added: "I2C2"
- note added: "LEDs Safety switch"
- note added: "Power regulation"
- note added: "SPI Dual I2C Dual CAN Aux ADC ports"
- note added: "Timer allocation: PE9: TIM1_CH1: FMU-CH4 PE11: TIM1_CH2: FMU-CH3 PE13: TIM1_CH3: FMU-CH2 PE14: TIM1_CH4: FMU-CH1 PA1: TIM5_CH2: FMU-CH7 PA2: TIM5_CH3: FMU-CH9 (NC) PA3: TIM5_CH4: FMU-CH10 (NC) PA15: TIM2_CH1: ALARM PB0: TIM3_CH3: GYRO1_DRDY PB1: TIM3_CH4: GYRO2_DRDY PB4: TIM3_CH1: ACCEL_DRDY PB5: TIM3_CH2: MAG_DRDY PD13: TIM4_CH2: FMU-CH5 PD14: TIM4_CH3: FMU-CH8 PD15: TIM4_CH4: FMU-CH6"
- note added: "USB Flash SWD Debug connector"
- note removed: "1206L150/12SL littlefuse"
- note removed: "Current Limits: I(limit) = 25000 / R(ilim) 25K = 1A, 16K5 = 1.5A"
- note removed: "FMU Power and Reset"
- note removed: "FMU Serial ports"
- note removed: "FMU SoC Ports FRAM"
- note removed: "LEDs Piezo driver Safety switch"
- note removed: "Peripherals Power Supply"
- note removed: "Power source selector"
- note removed: "SERIAL4"
- note removed: "SPI I2C Analog pressure CAN Aux ADC ports"
- note removed: "Timer allocation: PE9: TIM1_CH1: FMU-CH4 PE11: TIM1_CH2: FMU-CH3 PE13: TIM1_CH3: FMU-CH2 PE14: TIM1_CH4: FMU-CH1 PA15: TIM2_CH1: ALARM PB0: TIM3_CH3: GYRO1_DRDY PB1: TIM3_CH4: GYRO2_DRDY PB4: TIM3_CH1: ACCEL_DRDY PB5: TIM3_CH2: MAG_DRDY PD13: TIM4_CH2: FMU-CH5 PD14: TIM4_CH3: FMU-CH6 PD15: TIM4_CH4: spare"
- note removed: "USB Flash Expansion"

Commit message: Some uNode first layout
Parts:
- removed D701: MSS1P4-M3, pixhawk2:DIODE-SCHOTTKY_MSMP
- removed D901: (no value), SparkFun-DiscreteSemi:DIODESOD
- added D1, D2: DIODE-SCHOTTKY, SparkFun-DiscreteSemi:DIODE-SCHOTTKY
Connections:
- net FMU-CH1: now also L1001G$8.P$1; no longer L1001G$1.P$1
- net FMU-CH1-PROT: now also L1001G$8.P$2; no longer L1001G$1.P$2
- net FMU-CH2: now also L1001G$7.P$1; no longer L1001G$2.P$1
- net FMU-CH3: now also L1001G$6.P$1; no longer L1001G$3.P$1
- net FMU-CH4: now also L1001G$5.P$1; no longer L1001G$4.P$1
- net FMU-CH5: now also L1001G$4.P$1; no longer L1001G$5.P$1
- net FMU-CH6: now also L1001G$3.P$1; no longer L1001G$6.P$1
- net FMU-CH7: now also L1001G$2.P$1; no longer L1001G$7.P$1
- net FMU-CH8: now also L1001G$1.P$1; no longer L1001G$8.P$1
- net FMU-VDD_3V3: now also D2.A; no longer D701.A
- net GND: now also D1.A; no longer D901.A
- net N$15: now also L1001G$1.P$2; no longer L1001G$8.P$2
- net N$16: now also L1001G$2.P$2; no longer L1001G$7.P$2
- net N$36: now also L1001G$3.P$2; no longer L1001G$6.P$2
- net N$6: now also D1.C; no longer D901.C
- net N$68: now also L1001G$4.P$2; no longer L1001G$5.P$2
- net N$77: now also L1001G$5.P$2; no longer L1001G$4.P$2
- net N$78: now also L1001G$6.P$2; no longer L1001G$3.P$2
- net N$79: now also L1001G$7.P$2; no longer L1001G$2.P$2
- net N$9: now also D2.C; no longer D701.C
Other:
- moved on the sheet: L1001G$1, L1001G$2, L1001G$3, L1001G$4, L1001G$5, L1001G$6, L1001G$7, L1001G$8
Changed lines of the file:
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@@
 <attribute name="PARTNO" value="MSS1P4-M3/89A"/>
 </part>
-<part name="D901" library="SparkFun-DiscreteSemi" deviceset="DIODE" device="SOD">
-<attribute name="BOM" value="EXCLUDE"/>
-</part>
 <part name="D902" library="SparkFun-DiscreteSemi" deviceset="DIODE" device="SMA" value="B340A">
 <attribute name="PARTNO" value="B340A"/>
@@
 <part name="GND19" library="pixhawk2" deviceset="GND" device=""/>
 <part name="GND22" library="pixhawk2" deviceset="GND" device=""/>
-<part name="D701" library="pixhawk2" deviceset="DIODE-SCHOTTKY" device="_MSMP" value="MSS1P4-M3">
-<attribute name="PARTNO" value="MSS1P4-M3/89A"/>
-</part>
 <part name="JP1001" library="SparkFun-Connectors" deviceset="M01" device="SMD-4.5X1.5">
 <attribute name="BOM" value="EXCLUDE"/>
@@
 <part name="JP1" library="SparkFun-Connectors" deviceset="M03X2" device="2X3_SILK_SM"/>
 <part name="JP2" library="SparkFun-Connectors" deviceset="M03X2" device="2X3_SILK_SM"/>
+<part name="D1" library="SparkFun-DiscreteSemi" deviceset="DIODE-SCHOTTKY" device=""/>
+<part name="D2" library="SparkFun-DiscreteSemi" deviceset="DIODE-SCHOTTKY" device=""/>
 </parts>
 <sheets>
@@
 <attribute name="BOM" x="195.58" y="104.14" size="1.778" layer="96" display="off"/>
 </instance>
-<instance part="D701" gate="G$1" x="205.74" y="127" smashed="yes" rot="MR270">
-<attribute name="NAME" x="210.3374" y="127" size="1.778" layer="95" rot="MR270"/>
-<attribute name="PARTNO" x="205.74" y="127" size="1.778" layer="96" rot="MR90" display="off"/>
-</instance>
 <instance part="JP702" gate="G$1" x="195.58" y="91.44">
 <attribute name="BOM" x="195.58" y="91.44" size="1.778" layer="96" display="off"/>
 </instance>
+<instance part="D2" gate="G$1" x="205.74" y="127" rot="R270"/>
 </instances>
 <busses>
@@
 <label x="187.96" y="132.08" size="1.27" layer="95" rot="R180" xref="yes"/>
 <wire x1="223.52" y1="132.08" x2="205.74" y2="132.08" width="0.1524" layer="91"/>
-<pinref part="D701" gate="G$1" pin="A"/>
 <wire x1="205.74" y1="132.08" x2="187.96" y2="132.08" width="0.1524" layer="91"/>
 <wire x1="205.74" y1="129.54" x2="205.74" y2="132.08" width="0.1524" layer="91"/>
 <junction x="205.74" y="132.08"/>
+<pinref part="D2" gate="G$1" pin="A"/>
 </segment>
 <segment>
@@
 <segment>
 <pinref part="R706" gate="G$1" pin="2"/>
-<pinref part="D701" gate="G$1" pin="C"/>
 <wire x1="205.74" y1="121.92" x2="205.74" y2="124.46" width="0.1524" layer="91"/>
+<pinref part="D2" gate="G$1" pin="C"/>
 </segment>
 </net>
@@
 <attribute name="PARTNO" x="124.46" y="134.62" size="1.778" layer="96" rot="MR90" display="off"/>
 </instance>
-<instance part="D901" gate="G$1" x="81.28" y="86.36" rot="R90">
-<attribute name="BOM" x="81.28" y="86.36" size="1.778" layer="96" rot="R90" display="off"/>
-</instance>
 <instance part="D902" gate="G$1" x="104.14" y="127">
 <attribute name="PARTNO" x="104.14" y="127" size="1.778" layer="96" display="off"/>
@@
 </instance>
 <instance part="GND18" gate="1" x="78.74" y="144.78"/>
+<instance part="D1" gate="G$1" x="81.28" y="86.36" rot="R90"/>
 </instances>
 <busses>
@@
 <pinref part="R903" gate="G$1" pin="1"/>
 <wire x1="88.9" y1="68.58" x2="88.9" y2="71.12" width="0.1524" layer="91"/>
-<pinref part="D901" gate="G$1" pin="A"/>
 <wire x1="88.9" y1="71.12" x2="88.9" y2="73.66" width="0.1524" layer="91"/>
 <wire x1="88.9" y1="71.12" x2="81.28" y2="71.12" width="0.1524" layer="91"/>
 <wire x1="81.28" y1="71.12" x2="81.28" y2="83.82" width="0.1524" layer="91"/>
 <junction x="88.9" y="71.12"/>
+<pinref part="D1" gate="G$1" pin="A"/>
 </segment>
 <segment>
@@
 <net name="N$6" class="0">
 <segment>
-<pinref part="D901" gate="G$1" pin="C"/>
 <wire x1="81.28" y1="88.9" x2="81.28" y2="101.6" width="0.1524" layer="91"/>
 <pinref part="R902" gate="G$1" pin="2"/>
@@
 <wire x1="81.28" y1="101.6" x2="88.9" y2="101.6" width="0.1524" layer="91"/>
 <junction x="88.9" y="101.6"/>
+<pinref part="D1" gate="G$1" pin="C"/>
 </segment>
 </net>
@@
 <instances>
 <instance part="FRAME8" gate="G$1" x="0" y="0"/>
-<instance part="L1001" gate="G$1" x="81.28" y="99.06"/>
-<instance part="L1001" gate="G$2" x="68.58" y="104.14"/>
-<instance part="L1001" gate="G$3" x="53.34" y="109.22"/>
-<instance part="L1001" gate="G$4" x="81.28" y="114.3"/>
-<instance part="L1001" gate="G$5" x="66.04" y="119.38"/>
-<instance part="L1001" gate="G$6" x="53.34" y="124.46"/>
-<instance part="L1001" gate="G$7" x="78.74" y="129.54"/>
-<instance part="L1001" gate="G$8" x="66.04" y="134.62"/>
+<instance part="L1001" gate="G$8" x="81.28" y="99.06"/>
+<instance part="L1001" gate="G$7" x="68.58" y="104.14"/>
+<instance part="L1001" gate="G$6" x="53.34" y="109.22"/>
+<instance part="L1001" gate="G$5" x="81.28" y="114.3"/>
+<instance part="L1001" gate="G$4" x="66.04" y="119.38"/>
+<instance part="L1001" gate="G$3" x="53.34" y="124.46"/>
+<instance part="L1001" gate="G$2" x="78.74" y="129.54"/>
+<instance part="L1001" gate="G$1" x="66.04" y="134.62"/>
 <instance part="GND5" gate="1" x="144.78" y="106.68"/>
 <instance part="L1001" gate="G$9" x="144.78" y="116.84"/>
@@
 <wire x1="40.64" y1="99.06" x2="76.2" y2="99.06" width="0.1524" layer="91"/>
 <label x="40.64" y="99.06" size="1.27" layer="95" rot="R180" xref="yes"/>
-<pinref part="L1001" gate="G$1" pin="P$1"/>
+<pinref part="L1001" gate="G$8" pin="P$1"/>
 </segment>
 </net>
@@
 <wire x1="40.64" y1="104.14" x2="63.5" y2="104.14" width="0.1524" layer="91"/>
 <label x="40.64" y="104.14" size="1.27" layer="95" rot="R180" xref="yes"/>
-<pinref part="L1001" gate="G$2" pin="P$1"/>
+<pinref part="L1001" gate="G$7" pin="P$1"/>
 </segment>
 </net>
@@
 <wire x1="40.64" y1="109.22" x2="48.26" y2="109.22" width="0.1524" layer="91"/>
 <label x="40.64" y="109.22" size="1.27" layer="95" rot="R180" xref="yes"/>
-<pinref part="L1001" gate="G$3" pin="P$1"/>
+<pinref part="L1001" gate="G$6" pin="P$1"/>
 </segment>
 </net>
@@
 <segment>
 <wire x1="71.12" y1="119.38" x2="99.06" y2="119.38" width="0.1524" layer="91"/>
-<pinref part="L1001" gate="G$5" pin="P$2"/>
+<pinref part="L1001" gate="G$4" pin="P$2"/>
 <pinref part="J1001" gate="-CH5" pin="S"/>
 </segment>
@@
 <net name="N$77" class="0">
 <segment>
-<pinref part="L1001" gate="G$4" pin="P$2"/>
+<pinref part="L1001" gate="G$5" pin="P$2"/>
 <wire x1="86.36" y1="114.3" x2="99.06" y2="114.3" width="0.1524" layer="91"/>
 <pinref part="J1001" gate="-CH4" pin="S"/>
@@
 <net name="N$78" class="0">
 <segment>
-<pinref part="L1001" gate="G$3" pin="P$2"/>
+<pinref part="L1001" gate="G$6" pin="P$2"/>
 <wire x1="58.42" y1="109.22" x2="99.06" y2="109.22" width="0.1524" layer="91"/>
 <pinref part="J1001" gate="-CH3" pin="S"/>
@@
 <net name="N$79" class="0">
 <segment>
-<pinref part="L1001" gate="G$2" pin="P$2"/>
+<pinref part="L1001" gate="G$7" pin="P$2"/>
 <wire x1="73.66" y1="104.14" x2="99.06" y2="104.14" width="0.1524" layer="91"/>
 <pinref part="J1001" gate="-CH2" pin="S"/>
@@
 <net name="FMU-CH1-PROT" class="0">
 <segment>
-<pinref part="L1001" gate="G$1" pin="P$2"/>
+<pinref part="L1001" gate="G$8" pin="P$2"/>
 <wire x1="86.36" y1="99.06" x2="99.06" y2="99.06" width="0.1524" layer="91"/>
 <pinref part="J1001" gate="-CH1" pin="S"/>
@@
 <wire x1="40.64" y1="114.3" x2="76.2" y2="114.3" width="0.1524" layer="91"/>
 <label x="40.64" y="114.3" size="1.27" layer="95" rot="R180" xref="yes"/>
-<pinref part="L1001" gate="G$4" pin="P$1"/>
+<pinref part="L1001" gate="G$5" pin="P$1"/>
 </segment>
 </net>
@@
 <wire x1="40.64" y1="119.38" x2="60.96" y2="119.38" width="0.1524" layer="91"/>
 <label x="40.64" y="119.38" size="1.27" layer="95" rot="R180" xref="yes"/>
-<pinref part="L1001" gate="G$5" pin="P$1"/>
+<pinref part="L1001" gate="G$4" pin="P$1"/>
 </segment>
 </net>
@@
 <net name="N$15" class="0">
 <segment>
-<pinref part="L1001" gate="G$8" pin="P$2"/>
+<pinref part="L1001" gate="G$1" pin="P$2"/>
 <wire x1="71.12" y1="134.62" x2="99.06" y2="134.62" width="0.1524" layer="91"/>
 <pinref part="J1001" gate="-CH8" pin="S"/>
@@
 <segment>
 <wire x1="83.82" y1="129.54" x2="99.06" y2="129.54" width="0.1524" layer="91"/>
-<pinref part="L1001" gate="G$7" pin="P$2"/>
+<pinref part="L1001" gate="G$2" pin="P$2"/>
 <pinref part="J1001" gate="-CH7" pin="S"/>
 </segment>
@@
 <net name="N$36" class="0">
 <segment>
-<pinref part="L1001" gate="G$6" pin="P$2"/>
+<pinref part="L1001" gate="G$3" pin="P$2"/>
 <wire x1="58.42" y1="124.46" x2="99.06" y2="124.46" width="0.1524" layer="91"/>
 <pinref part="J1001" gate="-CH6" pin="S"/>
@@
 <wire x1="40.64" y1="134.62" x2="60.96" y2="134.62" width="0.1524" layer="91"/>
 <label x="40.64" y="134.62" size="1.27" layer="95" rot="R180" xref="yes"/>
-<pinref part="L1001" gate="G$8" pin="P$1"/>
+<pinref part="L1001" gate="G$1" pin="P$1"/>
 </segment>
 </net>
@@
 <segment>
 <label x="40.64" y="129.54" size="1.27" layer="95" rot="R180" xref="yes"/>
-<pinref part="L1001" gate="G$7" pin="P$1"/>
+<pinref part="L1001" gate="G$2" pin="P$1"/>
 <wire x1="40.64" y1="129.54" x2="73.66" y2="129.54" width="0.1524" layer="91"/>
 </segment>
@@
 <wire x1="40.64" y1="124.46" x2="48.26" y2="124.46" width="0.1524" layer="91"/>
 <label x="40.64" y="124.46" size="1.27" layer="95" rot="R180" xref="yes"/>
-<pinref part="L1001" gate="G$6" pin="P$1"/>
+<pinref part="L1001" gate="G$3" pin="P$1"/>
 </segment>
 </net>
