File: PX4uNode_V0_1_3.brd (EAGLE design)
At the start: 45.4 x 34 mm, 133 parts, among them J401 M04X2, M3_MOUNT1101 MOUNT-HOLE3.1MM, M3_MOUNT1102 MOUNT-HOLE3.1MM, M3_MOUNT1103 MOUNT-HOLE3.1MM, M3_MOUNT1104 MOUNT-HOLE3.1MM, U101 STM32F4X7VX, U401 MAX3051, U402 MAX3051, X101 3.2x2.5 mm / 24 MHz / 30 ppm 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

Commit message: Added PX4uNode_V01_01_3
Parts:
- added TP1, TP2, TP3, TP4, TP5: TPTP20R, testpad:TP20R
- moved JP1102 3.98 mm to (36.8, 31.9)
- moved R704 0.64 mm to (30.2, 31.4)
Connections:
- net FMU-!RESET: now also TP4.TP
- net FMU-SWCLK: now also TP2.TP
- net FMU-SWDIO: now also TP1.TP
- net FMU-SWO: now also TP3.TP
- net FMU-VDD_3V3: now also TP5.TP
- net GND: now also L403.P$1, L403.P$11, L403.P$12, L403.P$14, L403.P$16, L403.P$3, L403.P$5, L403.P$6
Routing:
- net VDD_SERVO_SENSE: track 22.6 -> 26.3 mm
- net FMU-SWO: track 5.87 -> 9.09 mm
- net GND: track 239.1 -> 241.9 mm, vias 41 -> 40
- net FMU-SWCLK: track 7.79 -> 10.5 mm
- net FMU-!RESET: track 37.0 -> 38.6 mm
- net FMU-SWDIO: track 10.2 -> 11.7 mm
- net FMU-VDD_3V3: track 81.2 -> 82.6 mm
