File: PX4uNode_V0_2_1.brd (EAGLE design)
At the start: 45.4 x 34 mm, 138 parts, among them J401 M04X2, M3_MOUNT1101 MOUNT-HOLE3.1MM, M3_MOUNT1102 MOUNT-HOLE3.1MM, M3_MOUNT1103 MOUNT-HOLE3.1MM, M3_MOUNT1104 MOUNT-HOLE3.1MM, U101 STM32F4X7VX, U401 MAX3051, U402 MAX3051, X101 3.2x2.5 mm / 24 MHz / 30 ppm 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

Commit message: Added PX4uNode_v0_2_1 files
Parts:
- moved TP5 19.5 mm to (28.3, 16.7)
- moved JP1102 1.74 mm to (38.5, 32.1)
- moved JP1104 1.69 mm to (41.4, 35.3)
- moved TP3 1.31 mm to (28.2, 20.0)
- moved JP1101 0.78 mm to (24.9, 10.1)
- moved D901 0.48 mm to (43.9, 33.8)
Connections:
- net !FRAM_CS: now also U$302.1
- net FMU-VDD_3V3: now also U$302.3, U$302.7
- net FRAM_MISO: now also U$302.2
- net FRAM_MOSI: now also U$302.5
- net FRAM_SCK: now also U$302.6
- net SDIO_CK: no longer U$302.6
- net SDIO_CMD: no longer U$302.1
- net SDIO_D0: no longer U$302.5
- net SDIO_D1: no longer U$302.2
- net SDIO_D2: no longer U$302.3
- net SDIO_D3: no longer U$302.7
Routing:
- net FRAM_MISO: track 0.00 -> 35.1 mm, vias 0 -> 3
- net !FRAM_CS: track 0.00 -> 33.8 mm, vias 0 -> 4
- net FRAM_SCK: track 0.00 -> 24.8 mm, vias 0 -> 2
- net SDIO_D2: track 22.4 -> 0.00 mm, vias 3 -> 0
- net SDIO_D1: track 20.8 -> 0.00 mm, vias 2 -> 0
- net FRAM_MOSI: track 0.00 -> 20.3 mm, vias 0 -> 3
- net SDIO_D0: track 15.2 -> 0.00 mm, vias 3 -> 0
- net SDIO_CMD: track 12.3 -> 0.00 mm
- net FMU-VDD_3V3: track 82.6 -> 91.3 mm, vias 22 -> 23
- net GND: track 241.9 -> 249.6 mm, vias 40 -> 44
- net SDIO_D3: track 5.87 -> 0.00 mm
- net FMU-USART3_RX: track 44.8 -> 50.5 mm
- net SDIO_CK: track 4.71 -> 0.00 mm
- net FMU-I2C2_SDA: track 25.0 -> 29.6 mm
- net FMU-USART3_RTS: track 37.5 -> 41.6 mm
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- added copper zone on layer 16, net 5V_S3_FILTERED
